File: hardware/remote-connector.kicad_pcb (KiCad board)
At the start: 2 copper layers, 10 x 7.8 mm, 6 parts, among them J1 Conn_01x03

Commit message: update universal connector pcb
Routing:
- net (no net): track 6.22 -> 7.58 mm
Changed lines of the file:
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@@
     (thickness 1)
     (drawings 7)
-    (tracks 15)
+    (tracks 20)
     (zones 0)
     (modules 6)
@@
       (usegerberadvancedattributes true)
       (creategerberjobfile true)
-      (excludeedgelayer false)
+      (excludeedgelayer true)
       (linewidth 0.100000)
       (plotframeref false)
@@
       (effects (font (size 1 1) (thickness 0.15)))
     )
+    (fp_line (start 2.45 1.12) (end -2.45 1.12) (layer F.CrtYd) (width 0.05))
+    (fp_line (start 2.45 -1.12) (end 2.45 1.12) (layer F.CrtYd) (width 0.05))
+    (fp_line (start -2.45 -1.12) (end 2.45 -1.12) (layer F.CrtYd) (width 0.05))
+    (fp_line (start -2.45 1.12) (end -2.45 -1.12) (layer F.CrtYd) (width 0.05))
+    (fp_line (start -0.727064 0.91) (end 0.727064 0.91) (layer F.SilkS) (width 0.12))
+    (fp_line (start -0.727064 -0.91) (end 0.727064 -0.91) (layer F.SilkS) (width 0.12))
+    (fp_line (start 1.6 0.8) (end -1.6 0.8) (layer F.Fab) (width 0.1))
+    (fp_line (start 1.6 -0.8) (end 1.6 0.8) (layer F.Fab) (width 0.1))
+    (fp_line (start -1.6 -0.8) (end 1.6 -0.8) (layer F.Fab) (width 0.1))
     (fp_line (start -1.6 0.8) (end -1.6 -0.8) (layer F.Fab) (width 0.1))
-    (fp_line (start -1.6 -0.8) (end 1.6 -0.8) (layer F.Fab) (width 0.1))
-    (fp_line (start 1.6 -0.8) (end 1.6 0.8) (layer F.Fab) (width 0.1))
-    (fp_line (start 1.6 0.8) (end -1.6 0.8) (layer F.Fab) (width 0.1))
-    (fp_line (start -0.727064 -0.91) (end 0.727064 -0.91) (layer F.SilkS) (width 0.12))
-    (fp_line (start -0.727064 0.91) (end 0.727064 0.91) (layer F.SilkS) (width 0.12))
-    (fp_line (start -2.45 1.12) (end -2.45 -1.12) (layer F.CrtYd) (width 0.05))
-    (fp_line (start -2.45 -1.12) (end 2.45 -1.12) (layer F.CrtYd) (width 0.05))
-    (fp_line (start 2.45 -1.12) (end 2.45 1.12) (layer F.CrtYd) (width 0.05))
-    (fp_line (start 2.45 1.12) (end -2.45 1.12) (layer F.CrtYd) (width 0.05))
     (fp_text user %R (at 0 0 90) (layer F.Fab)
       (effects (font (size 0.8 0.8) (thickness 0.12)))
@@
     (pad 2 smd roundrect (at 1.55 0 90) (size 1.3 1.75) (layers F.Cu F.Paste F.Mask) (roundrect_rratio 0.192)
       (net 3 "Net-(J1-Pad1)"))
-    (pad 1 smd roundrect (at -1.55 0 90) (size 1.3 1.75) (layers F.Cu F.Paste F.Mask) (roundrect_rratio 0.192308))
+    (pad 1 smd roundrect (at -1.55 0 90) (size 1.3 1.75) (layers F.Cu F.Paste F.Mask) (roundrect_rratio 0.1923076923076923))
     (model ${KISYS3DMOD}/Resistor_SMD.3dshapes/R_1206_3216Metric.wrl
       (at (xyz 0 0 0))
@@
   (module Connector_Wire:SolderWirePad_1x01_SMD_1x2mm (layer F.Cu)
     (at 22.7584 25.781 90)
+    (descr "Wire Pad, Square, SMD Pad,  5mm x 10mm,")
+    (tags "MesurementPoint Square SMDPad 5mmx10mm ")
+    (attr virtual)
+    (fp_text reference REF** (at 0 -2.54 90) (layer F.SilkS)
+      (effects (font (size 1 1) (thickness 0.15)))
+    )
+    (fp_text value SolderWirePad_1x01_SMD_1x2mm (at 0 2.54 90) (layer F.Fab)
+      (effects (font (size 1 1) (thickness 0.15)))
+    )
+    (fp_line (start -0.63 1.27) (end -0.63 -1.27) (layer F.Fab) (width 0.1))
+    (fp_line (start 0.63 1.27) (end -0.63 1.27) (layer F.Fab) (width 0.1))
+    (fp_line (start 0.63 -1.27) (end 0.63 1.27) (layer F.Fab) (width 0.1))
+    (fp_line (start -0.63 -1.27) (end 0.63 -1.27) (layer F.Fab) (width 0.1))
+    (fp_line (start -0.63 -1.27) (end -0.63 1.27) (layer F.CrtYd) (width 0.05))
+    (fp_line (start -0.63 1.27) (end 0.63 1.27) (layer F.CrtYd) (width 0.05))
+    (fp_line (start 0.63 1.27) (end 0.63 -1.27) (layer F.CrtYd) (width 0.05))
+    (fp_line (start 0.63 -1.27) (end -0.63 -1.27) (layer F.CrtYd) (width 0.05))
+    (fp_text user %R (at 0 0 90) (layer F.Fab)
+      (effects (font (size 1 1) (thickness 0.15)))
+    )
+    (pad 4 smd roundrect (at 0 0.019 90) (size 1 2) (layers F.Cu F.Paste F.Mask) (roundrect_rratio 0.25)
+      (net 1 "Net-(J1-Pad3)"))
+  )
+  (module Connector_Wire:SolderWirePad_1x01_SMD_1x2mm (layer F.Cu)
+    (at 22.7584 20.0152 90)
     (descr "Wire Pad, Square, SMD Pad,  5mm x 10mm,")
     (tags "MesurementPoint Square SMDPad 5mmx10mm ")
@@
       (effects (font (size 1 1) (thickness 0.15)))
     )
-    (pad 4 smd roundrect (at 0 0.019 90) (size 1 2) (layers F.Cu F.Paste F.Mask) (roundrect_rratio 0.25)
-      (net 1 "Net-(J1-Pad3)"))
+    (pad 1 smd roundrect (at 0 -0.0318 90) (size 1 2) (layers F.Cu F.Paste F.Mask) (roundrect_rratio 0.25)
+      (net 3 "Net-(J1-Pad1)"))
   )
   (module Connector_Wire:SolderWirePad_1x01_SMD_1x2mm (layer F.Cu)
-    (at 22.7584 20.0152 90)
+    (at 22.7584 21.997133 90)
     (descr "Wire Pad, Square, SMD Pad,  5mm x 10mm,")
     (tags "MesurementPoint Square SMDPad 5mmx10mm ")
@@
       (effects (font (size 1 1) (thickness 0.15)))
     )
-    (pad 1 smd roundrect (at 0 -0.0318 90) (size 1 2) (layers F.Cu F.Paste F.Mask) (roundrect_rratio 0.25)
-      (net 3 "Net-(J1-Pad1)"))
+    (pad 2 smd roundrect (at 0 -0.0064 90) (size 1 2) (layers F.Cu F.Paste F.Mask) (roundrect_rratio 0.25)
+      (net 2 "Net-(J1-Pad2)"))
   )
   (module Connector_Wire:SolderWirePad_1x01_SMD_1x2mm (layer F.Cu)
-    (at 22.7584 21.997133 90)
+    (at 22.7584 23.876 90)
     (descr "Wire Pad, Square, SMD Pad,  5mm x 10mm,")
     (tags "MesurementPoint Square SMDPad 5mmx10mm ")
@@
       (effects (font (size 1 1) (thickness 0.15)))
     )
-    (pad 2 smd roundrect (at 0 -0.0064 90) (size 1 2) (layers F.Cu F.Paste F.Mask) (roundrect_rratio 0.25)
-      (net 2 "Net-(J1-Pad2)"))
-  )
-  (module Connector_Wire:SolderWirePad_1x01_SMD_1x2mm (layer F.Cu)
-    (at 22.7584 23.876 90)
-    (descr "Wire Pad, Square, SMD Pad,  5mm x 10mm,")
-    (tags "MesurementPoint Square SMDPad 5mmx10mm ")
-    (attr virtual)
-    (fp_text reference REF** (at 0 -2.54 90) (layer F.SilkS)
-      (effects (font (size 1 1) (thickness 0.15)))
-    )
-    (fp_text value SolderWirePad_1x01_SMD_1x2mm (at 0 2.54 90) (layer F.Fab)
-      (effects (font (size 1 1) (thickness 0.15)))
-    )
-    (fp_line (start -0.63 1.27) (end -0.63 -1.27) (layer F.Fab) (width 0.1))
-    (fp_line (start 0.63 1.27) (end -0.63 1.27) (layer F.Fab) (width 0.1))
-    (fp_line (start 0.63 -1.27) (end 0.63 1.27) (layer F.Fab) (width 0.1))
-    (fp_line (start -0.63 -1.27) (end 0.63 -1.27) (layer F.Fab) (width 0.1))
-    (fp_line (start -0.63 -1.27) (end -0.63 1.27) (layer F.CrtYd) (width 0.05))
-    (fp_line (start -0.63 1.27) (end 0.63 1.27) (layer F.CrtYd) (width 0.05))
-    (fp_line (start 0.63 1.27) (end 0.63 -1.27) (layer F.CrtYd) (width 0.05))
-    (fp_line (start 0.63 -1.27) (end -0.63 -1.27) (layer F.CrtYd) (width 0.05))
-    (fp_text user %R (at 0 0 90) (layer F.Fab)
-      (effects (font (size 1 1) (thickness 0.15)))
-    )
     (pad 4 smd roundrect (at -0.103066 0.019 90) (size 1 2) (layers F.Cu F.Paste F.Mask) (roundrect_rratio 0.25))
   )
@@
       (effects (font (size 1 1) (thickness 0.15)))
     )
+    (fp_line (start -2.826861 -3) (end -2.826861 3.81) (layer Dwgs.User) (width 0.12))
+    (fp_line (start -2.826861 3.81) (end 4.858369 3.81) (layer Dwgs.User) (width 0.12))
+    (fp_line (start 4.858369 3.81) (end 4.858369 -3) (layer Dwgs.User) (width 0.12))
     (fp_line (start 4.858369 -3) (end -2.826861 -3) (layer Dwgs.User) (width 0.12))
-    (fp_line (start 4.858369 3.81) (end 4.858369 -3) (layer Dwgs.User) (width 0.12))
-    (fp_line (start -2.826861 3.81) (end 4.858369 3.81) (layer Dwgs.User) (width 0.12))
-    (fp_line (start -2.826861 -3) (end -2.826861 3.81) (layer Dwgs.User) (width 0.12))
     (pad 4 smd rect (at 4 -1.27 270) (size 1.1 3) (layers F.Cu F.Paste F.Mask)
       (net 1 "Net-(J1-Pad3)"))
@@
   (segment (start 29.760734 23.979066) (end 29.8196 23.9202) (width 0.4) (layer F.Cu) (net 0))
   (segment (start 29.735334 24.004466) (end 29.8196 23.9202) (width 0.4) (layer F.Cu) (net 0))
-  (segment (start 23.7172 24.004466) (end 29.735334 24.004466) (width 0.4) (layer F.Cu) (net 0))
+  (segment (start 29.8196 23.9202) (end 27.4762 23.9202) (width 0.4) (layer F.Cu) (net 0))
+  (segment (start 27.103 23.547) (end 25.0698 23.547) (width 0.4) (layer F.Cu) (net 0))
+  (segment (start 27.4762 23.9202) (end 27.103 23.547) (width 0.4) (layer F.Cu) (net 0))
+  (segment (start 24.637734 23.979066) (end 25.0698 23.547) (width 0.4) (layer F.Cu) (net 0))
+  (segment (start 22.7774 23.979066) (end 24.637734 23.979066) (width 0.4) (layer F.Cu) (net 0))
   (segment (start 29.6804 25.781) (end 29.8196 25.9202) (width 0.4) (layer F.Cu) (net 1))
   (segment (start 29.7058 25.8064) (end 29.8196 25.9202) (width 0.4) (layer F.Cu) (net 1))
@@
   (segment (start 24.638 20.0152) (end 25.0698 20.447) (width 0.4) (layer F.Cu) (net 3))
   (segment (start 22.7266 20.0152) (end 24.638 20.0152) (width 0.4) (layer F.Cu) (net 3))
-  (segment (start 25.5966 19.9202) (end 25.0698 20.447) (width 0.4) (layer F.Cu) (net 3))
-  (segment (start 29.8196 19.9202) (end 25.5966 19.9202) (width 0.4) (layer F.Cu) (net 3))
+  (segment (start 25.0698 20.447) (end 26.67 20.447) (width 0.4) (layer F.Cu) (net 3))
+  (segment (start 27.1968 19.9202) (end 29.8196 19.9202) (width 0.4) (layer F.Cu) (net 3))
+  (segment (start 26.67 20.447) (end 27.1968 19.9202) (width 0.4) (layer F.Cu) (net 3))
 )
